File: Design/ControlStage/LinearRegulator.sch (KiCad schematic (older format))
At the start: 24 parts, among them U3 LT3081_TO-220, U4 LT3081_TO-220

Commit message: Add files via upload
Parts:
- U3, U4: footprint Package_TO_SOT_THT:TO-220F-7_P2.54x3.7mm_StaggerEven_Lead3.5mm_Vertical -> Package_TO_SOT_THT:TO-220F-7_P2.54x3.7mm_StaggerOdd_Lead3.5mm_Vertical
Changed lines of the file:
@@
 Sheet 4 7
 Title "YAPS - Regulated Power Supply"
-Date "2019-05-26"
-Rev "0.1"
+Date "2019-06-08"
+Rev "1.1"
 Comp "Andrew Johnson"
 Comment1 ""
@@
 F 0 "U4" H 6100 2765 50  0000 C CNN
 F 1 "LT3081_TO-220" H 6100 2674 50  0000 C CNN
-F 2 "Package_TO_SOT_THT:TO-220F-7_P2.54x3.7mm_StaggerEven_Lead3.5mm_Vertical" H 5900 2100 50  0001 C CNN
+F 2 "Package_TO_SOT_THT:TO-220F-7_P2.54x3.7mm_StaggerOdd_Lead3.5mm_Vertical" H 5900 2100 50  0001 C CNN
 F 3 "http://www.linear.com/docs/43256" H 5900 2100 50  0001 C CNN
 F 4 "LT3081ET7#PBF-ND" H 6100 2250 50  0001 C CNN "Digikey Code"
@@
 F 0 "U3" H 6050 5015 50  0000 C CNN
 F 1 "LT3081_TO-220" H 6050 4924 50  0000 C CNN
-F 2 "Package_TO_SOT_THT:TO-220F-7_P2.54x3.7mm_StaggerEven_Lead3.5mm_Vertical" H 5850 4350 50  0001 C CNN
+F 2 "Package_TO_SOT_THT:TO-220F-7_P2.54x3.7mm_StaggerOdd_Lead3.5mm_Vertical" H 5850 4350 50  0001 C CNN
 F 3 "http://www.linear.com/docs/43256" H 5850 4350 50  0001 C CNN
 F 4 "LT3081ET7#PBF-ND" H 6050 4500 50  0001 C CNN "Digikey Code"
