File: Design/ControlStage/LowVoltageSupply.sch (KiCad schematic (older format))
At the start: 3 parts, among them U7 LM7805_TO220

Commit message: Add files via upload
Parts:
- removed C27: 0.33uF, Capacitor_SMD:C_0805_2012Metric_Pad1.15x1.40mm_HandSolder, symbol Device:C
- removed C28: 0.1uF, Resistor_SMD:R_0805_2012Metric_Pad1.15x1.40mm_HandSolder, symbol Device:C
- U7: value LM7805_TO220 -> TSR1-2450; footprint Package_TO_SOT_THT:TO-220-3_Vertical -> CustomFootprintLibrary:TSR1-24xx_TO-220-3; symbol Regulator_Linear:LM7805_TO220 -> CustomSymbolLibrary:TSR1-24xx; Farnell Code 2323602 -> (none); RS Code (none) -> 666-4379
Other:
- note added: "Also use:\nTSR1N 1-2450 Farnell Code 2323602\nLM7805: do thermal calc: Voltage drop * Current of Arduino used."
- note added: "If LM7805 used add:\n- 0.33uF capacitor from Vin to GND\n- 0.1uF capacitor from Vout to GND"
Changed lines of the file:
@@
 Sheet 7 7
 Title "YAPS - Regulated Power Supply"
-Date "2019-05-26"
-Rev "0.1"
+Date "2019-06-08"
+Rev "1.1"
 Comp "Andrew Johnson"
-Comment1 ""
+Comment1 "1.1 - changed UA7805 to TSR1-2450"
 Comment2 ""
 Comment3 ""
@@
 Text HLabel 1000 1000 0    50   Input ~ 0
 PI
-Wire Wire Line
-	1000 1000 1300 1000
 $Comp
-L Device:C C27
-U 1 1 5CAA62A2
-P 1300 1250
-F 0 "C27" H 1415 1296 50  0000 L CNN
-F 1 "0.33uF" H 1415 1205 50  0000 L CNN
-F 2 "Capacitor_SMD:C_0805_2012Metric_Pad1.15x1.40mm_HandSolder" H 1338 1100 50  0001 C CNN
-F 3 "http://www.farnell.com/datasheets/1901289.pdf?_ga=2.8331319.464475340.1555178862-441347304.1541859637&_gac=1.238225716.1554891125.EAIaIQobChMI16fD9tLD4QIVz5TtCh3QQglqEAAYAiAAEgKKrvD_BwE" H 1300 1250 50  0001 C CNN
-F 4 "2320844" H 1300 1250 50  0001 C CNN "Farnell Code"
-	1    1300 1250
+L CustomSymbolLibrary:TSR1-24xx U7
+U 1 1 5CAA760D
+P 2600 850
+F 0 "U7" H 2600 950 50  0000 C CNN
+F 1 "TSR1-2450" H 2600 850 50  0000 C CNN
+F 2 "CustomFootprintLibrary:TSR1-24xx_TO-220-3" H 2600 1075 50  0001 C CIN
+F 3 "https://docs-emea.rs-online.com/webdocs/16ed/0900766b816ed3dd.pdf" H 2600 800 50  0001 C CNN
+F 4 "666-4379" H 2600 850 50  0001 C CNN "RS Code"
+	1    2600 850
 	1    0    0    -1
 $EndComp
-Wire Wire Line
-	1300 1100 1300 1000
-Connection ~ 1300 1000
-Wire Wire Line
-	1300 1400 1300 1650
-$Comp
-L power:GNDPWR #PWR039
-U 1 1 5CAA69DB
-P 1300 1650
-F 0 "#PWR039" H 1300 1400 50  0001 C CNN
-F 1 "GNDPWR" H 1305 1477 50  0000 C CNN
-F 2 "" H 1300 1650 50  0001 C CNN
-F 3 "" H 1300 1650 50  0001 C CNN
-	1    1300 1650
-	1    0    0    -1
-$EndComp
-$Comp
-L Regulator_Linear:LM7805_TO220 U7
-U 1 1 5CAA760D
-P 2600 1000
-F 0 "U7" H 2600 1242 50  0000 C CNN
-F 1 "LM7805_TO220" H 2600 1151 50  0000 C CNN
-F 2 "Package_TO_SOT_THT:TO-220-3_Vertical" H 2600 1225 50  0001 C CIN
-F 3 "http://www.ti.com/general/docs/lit/getliterature.tsp?genericPartNumber=UA78&fileType=pdf" H 2600 950 50  0001 C CNN
-F 4 "2323602" H 2600 1000 50  0001 C CNN "Farnell Code"
-	1    2600 1000
-	1    0    0    -1
-$EndComp
-Wire Wire Line
-	2600 1300 2600 1650
 $Comp
 L power:GNDPWR #PWR040
@@
 	1    0    0    -1
 $EndComp
-$Comp
-L Device:C C28
-U 1 1 5CAAB531
-P 3200 1250
-F 0 "C28" H 3315 1296 50  0000 L CNN
-F 1 "0.1uF" H 3315 1205 50  0000 L CNN
-F 2 "Resistor_SMD:R_0805_2012Metric_Pad1.15x1.40mm_HandSolder" H 3238 1100 50  0001 C CNN
-F 3 "http://www.farnell.com/datasheets/1901289.pdf?_ga=2.217959571.464475340.1555178862-441347304.1541859637&_gac=1.205178532.1554891125.EAIaIQobChMI16fD9tLD4QIVz5TtCh3QQglqEAAYAiAAEgKKrvD_BwE" H 3200 1250 50  0001 C CNN
-F 4 "2320839" H 3200 1250 50  0001 C CNN "Farnell Code"
-	1    3200 1250
-	1    0    0    -1
-$EndComp
-Wire Wire Line
-	3200 1100 3200 1000
-Wire Wire Line
-	3200 1400 3200 1650
-$Comp
-L power:GNDPWR #PWR041
-U 1 1 5CAAB539
-P 3200 1650
-F 0 "#PWR041" H 3200 1400 50  0001 C CNN
-F 1 "GNDPWR" H 3205 1477 50  0000 C CNN
-F 2 "" H 3200 1650 50  0001 C CNN
-F 3 "" H 3200 1650 50  0001 C CNN
-	1    3200 1650
-	1    0    0    -1
-$EndComp
-Wire Wire Line
-	2900 1000 3200 1000
-Connection ~ 3200 1000
 Text HLabel 4300 1000 2    50   Input ~ 0
 REG_5v
 Wire Wire Line
-	1300 1000 2300 1000
+	2600 1350 2600 1650
+Text Notes 2950 800  0    50   ~ 0
+Also use:\nTSR1N 1-2450 Farnell Code 2323602\nLM7805: do thermal calc: Voltage drop * Current of Arduino used.
+Text Notes 850  2300 0    50   ~ 0
+If LM7805 used add:\n- 0.33uF capacitor from Vin to GND\n- 0.1uF capacitor from Vout to GND
 Wire Wire Line
-	3200 1000 4300 1000
+	1000 1000 2300 1000
+Wire Wire Line
+	2900 1000 4300 1000
 $EndSCHEMATC
