File: Design/ControlStage/PowerSupply.kicad_pcb (KiCad board)
At the start: 2 copper layers, 100 x 75 mm, 72 parts, among them J1 Conn_01x02, J2 Conn_01x02, J3 Conn_01x06, J4 Conn_01x08, J5 Conn_01x02, J6 Conn_01x06, Q1 IRF3205, Q2 2N3906, Q3 2N3904, U1 LTC1624CS8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

Commit message: Add files via upload
Parts:
- removed C27: 0.33uF, Capacitor_SMD:C_0805_2012Metric_Pad1.15x1.40mm_HandSolder
- removed C28: 0.1uF, Resistor_SMD:R_0805_2012Metric_Pad1.15x1.40mm_HandSolder
- Q2: footprint Package_TO_SOT_THT:TO-92_Inline -> CustomFootprintLibrary:TO-92_Inline_Wide
- U3, U4: footprint Package_TO_SOT_THT:TO-220F-7_P2.54x3.7mm_StaggerEven_Lead3.5mm_Vertical -> Package_TO_SOT_THT:TO-220F-7_P2.54x3.7mm_StaggerOdd_Lead3.5mm_Vertical
- U7: value LM7805_TO220 -> TSR1-2450; footprint Package_TO_SOT_THT:TO-220-3_Vertical -> CustomFootprintLibrary:TSR1-24xx_TO-220-3
- moved R10 9.14 mm to (145.9, 100.1)
- moved R12 6.50 mm to (140.0, 100.1), turned to 180 degrees
- moved U4 4.01 mm to (118.2, 106.5)
- moved U3 4.00 mm to (146.5, 106.5)
- moved U7 3.72 mm to (97.8, 58.5)
- moved R4 3.56 mm to (66.0, 95.0)
- moved Q2 3.54 mm to (75.0, 95.5), turned to 180 degrees
- moved R11 1.00 mm to (122.5, 109.0)
Routing:
- net /ON-OFF: track 105.3 -> 140.3 mm, vias 3 -> 4
- net /ICTRL+: track 71.2 -> 84.9 mm
- net /Linear Regulator 1/REGin: track 121.9 -> 111.5 mm
- net Net-(C4-Pad2): track 33.9 -> 29.6 mm
- net /T2OUT: track 45.9 -> 42.0 mm
- net Net-(C17-Pad1): track 39.1 -> 42.1 mm
- net Net-(C8-Pad2): track 12.7 -> 9.84 mm
- net VCC: track 70.9 -> 73.7 mm
- net /T1OUT: track 50.4 -> 48.1 mm
- net Net-(Q2-Pad2): track 13.6 -> 11.5 mm
- net /REG5V: track 135.9 -> 134.1 mm
- net Net-(R15-Pad2): track 43.8 -> 44.8 mm, vias 2 -> 1
- net /IMON: track 82.6 -> 83.4 mm
- net GNDS: vias 168 -> 175
- net GNDPWR: vias 33 -> 37
Other:
- board text added: "2019-06-08"
- board text added: "YAPS v1.1"
- board text removed: "2019-05-26"
- board text removed: "YAPS v1.0"
