File: Design/ControlStage/SwitchingRegulator.sch (KiCad schematic (older format))
At the start: 18 parts, among them Q1 IRF3205, Q2 2N3906, U1 LTC1624CS8

Commit message: Add files via upload
Parts:
- Q2: footprint Package_TO_SOT_THT:TO-92_Inline -> CustomFootprintLibrary:TO-92_Inline_Wide
Changed lines of the file:
@@
 Sheet 2 7
 Title "YAPS - Regulated Power Supply"
-Date "2019-05-26"
-Rev "0.1"
+Date "2019-06-08"
+Rev "1.1"
 Comp "Andrew Johnson"
 Comment1 ""
@@
 P 4600 3050
 F 0 "#PWR010" H 4600 2800 50  0001 C CNN
-F 1 "GNDS" H 4600 2700 50  0000 C CNN
+F 1 "GNDS" H 4600 2900 50  0000 C CNN
 F 2 "" H 4600 3050 50  0001 C CNN
 F 3 "" H 4600 3050 50  0001 C CNN
@@
 F 0 "Q2" H 6841 4354 50  0000 L CNN
 F 1 "2N3906" H 6841 4445 50  0000 L CNN
-F 2 "Package_TO_SOT_THT:TO-92_Inline" H 6850 4325 50  0001 L CIN
+F 2 "CustomFootprintLibrary:TO-92_Inline_Wide" H 6850 4325 50  0001 L CIN
 F 3 "https://www.onsemi.com/pub/Collateral/2N3906-D.PDF" H 6650 4400 50  0001 L CNN
 F 4 "2453753" H 6650 4400 50  0001 C CNN "Farnell Code"
