File: Design/PowerStage/PowerStage.kicad_pcb (KiCad board)
At the start: 2 copper layers, 96 x 56 mm, 6 parts, among them J1 Conn_01x02, J2 Conn_01x02

Commit message: Add files via upload
Parts:
- D1: footprint CustomFootprintLibrary:Diode_Bridge_23.0x3.5x10.0mm_P5.0mm -> CustomFootprintLibrary:Diode_Bridge_23.0x3.5mm_P5.0mm
- turned D1 to 0 degrees
Connections:
- D1 pad 1: +V -> 0V
- D1 pad 4: 0V -> +V
Routing:
- net Vac+: track 39.9 -> 43.6 mm
- net Vac-: vias 16 -> 17
- net 0V: vias 44 -> 62
Other:
- board text added: "2019-06-08"
- board text added: "AC"
- board text added: "YAPS v1.1"
- board text removed: "2019-05-26"
- board text removed: "YAPS v1.0"
